Commit message: fix: working barriers (both approaches)

File: examples/barriers/models/iiwa14_spheres_collision.urdf (robot description, URDF)
Before this commit: robot iiwa14, 19 links, 18 joints
Links:
- link first_iiwa_link_0: geometry collision sphere radius=0.15; visual mesh filename=package://examples/barriers/models/meshes/visual/link_0.obj
- link second_iiwa_link_0: geometry collision sphere radius=0.15; visual mesh filename=package://examples/barriers/models/meshes/visual/link_0.obj
